File: schematics/b1/initial_state_register.kicad_sch (KiCad schematic)
At the start: 20 parts, among them SW1 SW_SPDT, SW2 SW_SPDT, SW3 SW_SPDT, SW4 SW_SPDT, SW5 SW_SPDT, SW6 SW_SPDT, SW7 SW_SPDT, SW8 SW_Push, U1 74HC165

Commit message: General schematic updates.
Parts:
- removed SW1, SW2, SW3, SW4, SW5, SW6, SW7: SW_SPDT, symbol Switch:SW_SPDT
- removed SW8: SW_Push, symbol Switch:SW_Push
- added SW1: SW_DIP_x08, symbol Switch:SW_DIP_x08
- renumbered U1 to U2
Connections:
- net GND: now also R1.2, R2.2, R3.2, R4.2, R5.2, R6.2, R7.2, R8.2; no longer R1.1, R2.1, R3.1, R4.1, R5.1, R6.1, R7.1, R8.1
- net VCC: now also SW1.1, SW1.2, SW1.3, SW1.4, SW1.5, SW1.6, SW1.7, SW1.8
- net at U2.5 (D6): now also R7.1, SW1.10
- net at U2.12 (D1): now also R2.1, SW1.15
- net at U2.6 (D7): now also R8.1, SW1.9; no longer R8.2
- net at U2.11 (D0): now also R1.1, SW1.16
- net at U2.13 (D2): now also R3.1, SW1.14
- net at U2.4 (D5): now also R6.1, SW1.11
- net at U2.3 (D4): now also R5.1, SW1.12
- net at U2.14 (D3): now also R4.1, SW1.13
Other:
- note added: "Position 1 to 7 are switches that dictate the unit ID and are read upon startup. Position 8 is a reset switch and if it is high on boot, then EEPROM will be discarded."
- note removed: "SW1 to SW7 are DIP switches that dictate the unit ID and are read upon startup. SW8 is a momentary push button that, if high upon boot, will clear the EEPROM of the MCU."
- moved on the sheet: C1, C2, C3, U2
