File: schematics/b1/initial_state_register.kicad_sch (KiCad schematic)
At the start: 13 parts, among them SW1 SW_DIP_x08, U2 74HC165

Commit message: Resorted to bitbanging the status block blinkers.
Parts:
- removed C2: 1u, symbol Device:C
- C3: value 10u -> 1u
Other:
- moved on the sheet: C3
Changed lines of the file:
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@@
   (junction (at 85.09 63.5) (diameter 0) (color 0 0 0 0)
   )
-  (junction (at 156.21 41.91) (diameter 0) (color 0 0 0 0)
-  )
   (junction (at 73.66 82.55) (diameter 0) (color 0 0 0 0)
   )
@@
   )
   (junction (at 96.52 71.12) (diameter 0) (color 0 0 0 0)
-  )
-  (junction (at 144.78 31.75) (diameter 0) (color 0 0 0 0)
   )
   (junction (at 92.71 82.55) (diameter 0) (color 0 0 0 0)
@@
     (stroke (width 0) (type default))
   )
-  (wire (pts (xy 156.21 40.64) (xy 156.21 41.91))
-    (stroke (width 0) (type default))
-  )
   (wire (pts (xy 116.84 31.75) (xy 132.08 31.75))
     (stroke (width 0) (type default))
@@
     (stroke (width 0) (type default))
   )
-  (wire (pts (xy 144.78 41.91) (xy 156.21 41.91))
-    (stroke (width 0) (type default))
-  )
   (wire (pts (xy 69.85 53.34) (xy 69.85 73.66))
     (stroke (width 0) (type default))
@@
     (stroke (width 0) (type default))
   )
+  (wire (pts (xy 132.08 41.91) (xy 144.78 41.91))
+    (stroke (width 0) (type default))
+  )
   (wire (pts (xy 50.8 50.8) (xy 50.8 53.34))
     (stroke (width 0) (type default))
@@
     (stroke (width 0) (type default))
   )
+  (wire (pts (xy 92.71 82.55) (xy 96.52 82.55))
+    (stroke (width 0) (type default))
+  )
+  (wire (pts (xy 96.52 71.12) (xy 104.14 71.12))
+    (stroke (width 0) (type default))
+  )
+  (wire (pts (xy 50.8 58.42) (xy 52.07 58.42))
+    (stroke (width 0) (type default))
+  )
+  (wire (pts (xy 88.9 82.55) (xy 88.9 81.28))
+    (stroke (width 0) (type default))
+  )
+  (wire (pts (xy 67.31 58.42) (xy 77.47 58.42))
+    (stroke (width 0) (type default))
+  )
+  (wire (pts (xy 50.8 53.34) (xy 50.8 55.88))
+    (stroke (width 0) (type default))
+  )
+  (wire (pts (xy 88.9 66.04) (xy 88.9 73.66))
+    (stroke (width 0) (type default))
+  )
+  (wire (pts (xy 73.66 55.88) (xy 104.14 55.88))
+    (stroke (width 0) (type default))
+  )
+  (wire (pts (xy 144.78 43.18) (xy 144.78 41.91))
+    (stroke (width 0) (type default))
+  )
+  (wire (pts (xy 67.31 55.88) (xy 73.66 55.88))
+    (stroke (width 0) (type default))
+  )
+  (wire (pts (xy 116.84 31.75) (xy 116.84 43.18))
+    (stroke (width 0) (type default))
+  )
   (wire (pts (xy 132.08 31.75) (xy 144.78 31.75))
     (stroke (width 0) (type default))
   )
-  (wire (pts (xy 92.71 82.55) (xy 96.52 82.55))
-    (stroke (width 0) (type default))
-  )
-  (wire (pts (xy 96.52 71.12) (xy 104.14 71.12))
-    (stroke (width 0) (type default))
-  )
-  (wire (pts (xy 50.8 58.42) (xy 52.07 58.42))
-    (stroke (width 0) (type default))
-  )
-  (wire (pts (xy 88.9 82.55) (xy 88.9 81.28))
-    (stroke (width 0) (type default))
-  )
-  (wire (pts (xy 67.31 58.42) (xy 77.47 58.42))
-    (stroke (width 0) (type default))
-  )
-  (wire (pts (xy 50.8 53.34) (xy 50.8 55.88))
-    (stroke (width 0) (type default))
-  )
-  (wire (pts (xy 88.9 66.04) (xy 88.9 73.66))
-    (stroke (width 0) (type default))
-  )
-  (wire (pts (xy 73.66 55.88) (xy 104.14 55.88))
-    (stroke (width 0) (type default))
-  )
-  (wire (pts (xy 156.21 43.18) (xy 156.21 41.91))
-    (stroke (width 0) (type default))
-  )
-  (wire (pts (xy 144.78 41.91) (xy 132.08 41.91))
-    (stroke (width 0) (type default))
-  )
-  (wire (pts (xy 67.31 55.88) (xy 73.66 55.88))
-    (stroke (width 0) (type default))
-  )
-  (wire (pts (xy 116.84 31.75) (xy 116.84 43.18))
-    (stroke (width 0) (type default))
-  )
-  (wire (pts (xy 156.21 33.02) (xy 156.21 31.75))
-    (stroke (width 0) (type default))
-  )
   (wire (pts (xy 67.31 66.04) (xy 88.9 66.04))
     (stroke (width 0) (type default))
@@
   )
   (wire (pts (xy 67.31 68.58) (xy 92.71 68.58))
-    (stroke (width 0) (type default))
-  )
-  (wire (pts (xy 144.78 31.75) (xy 156.21 31.75))
     (stroke (width 0) (type default))
   )
@@
     )
   )
-  (symbol (lib_id "Device:C") (at 144.78 36.83 0) (unit 1)
-    (in_bom yes) (on_board yes) (dnp no) (fields_autoplaced)
-    (property "Reference" "C2" (at 148.59 35.56 0)
-      (effects (font (size 1.27 1.27)) (justify left))
-    )
-    (property "Value" "1u" (at 148.59 38.1 0)
-      (effects (font (size 1.27 1.27)) (justify left))
-    )
-    (property "Footprint" "" (at 145.7452 40.64 0)
-      (effects (font (size 1.27 1.27)) hide)
-    )
-    (property "Datasheet" "~" (at 144.78 36.83 0)
-      (effects (font (size 1.27 1.27)) hide)
-    )
-    (pin "2")
-    (pin "1")
-    (instances
-      (project "b1"
-        (path "/d6142fa5-2354-4512-9919-37616259c364/15951702-f191-4c4b-b68c-efdb5de618b5"
-          (reference "C2") (unit 1)
-        )
-      )
-    )
-  )
   (symbol (lib_id "Device:R") (at 88.9 77.47 0) (unit 1)
     (in_bom yes) (on_board yes) (dnp no)
@@
     )
   )
-  (symbol (lib_id "power:GND") (at 156.21 43.18 0) (unit 1)
+  (symbol (lib_id "power:GND") (at 144.78 43.18 0) (unit 1)
     (in_bom yes) (on_board yes) (dnp no) (fields_autoplaced)
-    (property "Reference" "#PWR025" (at 156.21 49.53 0)
-      (effects (font (size 1.27 1.27)) hide)
-    )
-    (property "Value" "GND" (at 156.21 48.26 0)
-      (effects (font (size 1.27 1.27)))
-    )
-    (property "Footprint" "" (at 156.21 43.18 0)
-      (effects (font (size 1.27 1.27)) hide)
-    )
-    (property "Datasheet" "" (at 156.21 43.18 0)
+    (property "Reference" "#PWR025" (at 144.78 49.53 0)
+      (effects (font (size 1.27 1.27)) hide)
+    )
+    (property "Value" "GND" (at 144.78 48.26 0)
+      (effects (font (size 1.27 1.27)))
+    )
+    (property "Footprint" "" (at 144.78 43.18 0)
+      (effects (font (size 1.27 1.27)) hide)
+    )
+    (property "Datasheet" "" (at 144.78 43.18 0)
       (effects (font (size 1.27 1.27)) hide)
     )
@@
     )
   )
-  (symbol (lib_id "Device:C_Polarized") (at 156.21 36.83 0) (unit 1)
+  (symbol (lib_id "Device:C_Polarized") (at 144.78 36.83 0) (unit 1)
     (in_bom yes) (on_board yes) (dnp no)
-    (property "Reference" "C3" (at 160.02 35.56 0)
+    (property "Reference" "C3" (at 148.59 35.56 0)
       (effects (font (size 1.27 1.27)) (justify left))
     )
-    (property "Value" "10u" (at 160.02 38.1 0)
+    (property "Value" "1u" (at 148.59 38.1 0)
       (effects (font (size 1.27 1.27)) (justify left))
     )
-    (property "Footprint" "" (at 157.1752 40.64 0)
-      (effects (font (size 1.27 1.27)) hide)
-    )
-    (property "Datasheet" "~" (at 156.21 36.83 0)
-      (effects (font (size 1.27 1.27)) hide)
-    )
+    (property "Footprint" "" (at 145.7452 40.64 0)
+      (effects (font (size 1.27 1.27)) hide)
+    )
+    (property "Datasheet" "~" (at 144.78 36.83 0)
+      (effects (font (size 1.27 1.27)) hide)
+    )

Commit message: Updated Wi-Fi block with a jumper switch as a workaround.
Parts:
- C3: symbol Device:C_Polarized -> Device:C
Changed lines of the file:
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@@
     )
   )
-  (symbol (lib_id "Device:C_Polarized") (at 144.78 36.83 0) (unit 1)
+  (symbol (lib_id "Device:C") (at 144.78 36.83 0) (unit 1)
     (in_bom yes) (on_board yes) (dnp no)
     (property "Reference" "C3" (at 148.59 35.56 0)

Commit message: Updated annotations.
Parts:
- renumbered C1 to C2, R5 to R10, R6 to R11, R7 to R12, R8 to R13, R1 to R6, R2 to R7, R3 to R8, R4 to R9, SW1 to SW4, U2 to U3
Changed lines of the file:
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@@
   (title_block
     (title "Initial State Register")
-    (date "2024-02-06")
+    (date "2024-02-15")
     (rev "1")
     (company "shawnd.xyz")
@@
   (symbol (lib_id "power:GND") (at 116.84 91.44 0) (unit 1)
     (in_bom yes) (on_board yes) (dnp no) (fields_autoplaced)
-    (property "Reference" "#PWR024" (at 116.84 97.79 0)
+    (property "Reference" "#PWR08" (at 116.84 97.79 0)
       (effects (font (size 1.27 1.27)) hide)
     )
@@
       (project "b1"
         (path "/d6142fa5-2354-4512-9919-37616259c364/15951702-f191-4c4b-b68c-efdb5de618b5"
-          (reference "#PWR024") (unit 1)
+          (reference "#PWR08") (unit 1)
         )
       )
@@
   (symbol (lib_id "Device:R") (at 92.71 77.47 0) (unit 1)
     (in_bom yes) (on_board yes) (dnp no)
-    (property "Reference" "R7" (at 92.71 85.09 0)
+    (property "Reference" "R12" (at 92.71 85.09 0)
       (effects (font (size 1.27 1.27)))
     )
@@
       (project "b1"
         (path "/d6142fa5-2354-4512-9919-37616259c364/15951702-f191-4c4b-b68c-efdb5de618b5"
-          (reference "R7") (unit 1)
+          (reference "R12") (unit 1)
         )
       )
@@
   (symbol (lib_id "Device:C") (at 132.08 36.83 0) (unit 1)
     (in_bom yes) (on_board yes) (dnp no) (fields_autoplaced)
-    (property "Reference" "C1" (at 135.89 35.56 0)
+    (property "Reference" "C2" (at 135.89 35.56 0)
       (effects (font (size 1.27 1.27)) (justify left))
     )
@@
       (project "b1"
         (path "/d6142fa5-2354-4512-9919-37616259c364/15951702-f191-4c4b-b68c-efdb5de618b5"
-          (reference "C1") (unit 1)
+          (reference "C2") (unit 1)
         )
       )
@@
   (symbol (lib_id "Switch:SW_DIP_x08") (at 59.69 63.5 0) (unit 1)
     (in_bom yes) (on_board yes) (dnp no) (fields_autoplaced)
-    (property "Reference" "SW1" (at 59.69 45.72 0)
+    (property "Reference" "SW4" (at 59.69 45.72 0)
       (effects (font (size 1.27 1.27)))
     )
@@
       (project "b1"
         (path "/d6142fa5-2354-4512-9919-37616259c364/15951702-f191-4c4b-b68c-efdb5de618b5"
-          (reference "SW1") (unit 1)
+          (reference "SW4") (unit 1)
         )
       )
@@
   (symbol (lib_id "Device:R") (at 85.09 77.47 0) (unit 1)
     (in_bom yes) (on_board yes) (dnp no)
-    (property "Reference" "R5" (at 85.09 85.09 0)
+    (property "Reference" "R10" (at 85.09 85.09 0)
       (effects (font (size 1.27 1.27)))
     )
@@
       (project "b1"
         (path "/d6142fa5-2354-4512-9919-37616259c364/15951702-f191-4c4b-b68c-efdb5de618b5"
-          (reference "R5") (unit 1)
+          (reference "R10") (unit 1)
         )
       )
@@
   (symbol (lib_id "Device:R") (at 96.52 77.47 0) (unit 1)
     (in_bom yes) (on_board yes) (dnp no)
-    (property "Reference" "R8" (at 96.52 85.09 0)
+    (property "Reference" "R13" (at 96.52 85.09 0)
       (effects (font (size 1.27 1.27)))
     )
@@
       (project "b1"
         (path "/d6142fa5-2354-4512-9919-37616259c364/15951702-f191-4c4b-b68c-efdb5de618b5"
-          (reference "R8") (unit 1)
+          (reference "R13") (unit 1)
         )
       )
@@
   (symbol (lib_id "Device:R") (at 88.9 77.47 0) (unit 1)
     (in_bom yes) (on_board yes) (dnp no)
-    (property "Reference" "R6" (at 88.9 85.09 0)
+    (property "Reference" "R11" (at 88.9 85.09 0)
       (effects (font (size 1.27 1.27)))
     )
@@
       (project "b1"
         (path "/d6142fa5-2354-4512-9919-37616259c364/15951702-f191-4c4b-b68c-efdb5de618b5"
-          (reference "R6") (unit 1)
+          (reference "R11") (unit 1)
         )
       )
@@
   (symbol (lib_id "power:GND") (at 144.78 43.18 0) (unit 1)
     (in_bom yes) (on_board yes) (dnp no) (fields_autoplaced)
-    (property "Reference" "#PWR025" (at 144.78 49.53 0)
+    (property "Reference" "#PWR09" (at 144.78 49.53 0)
       (effects (font (size 1.27 1.27)) hide)
     )
@@
       (project "b1"
         (path "/d6142fa5-2354-4512-9919-37616259c364/15951702-f191-4c4b-b68c-efdb5de618b5"
-          (reference "#PWR025") (unit 1)
+          (reference "#PWR09") (unit 1)
         )
       )
@@
   (symbol (lib_id "Device:R") (at 73.66 77.47 0) (unit 1)
     (in_bom yes) (on_board yes) (dnp no)
-    (property "Reference" "R2" (at 73.66 85.09 0)
+    (property "Reference" "R7" (at 73.66 85.09 0)
       (effects (font (size 1.27 1.27)))
     )
@@
       (project "b1"
         (path "/d6142fa5-2354-4512-9919-37616259c364/15951702-f191-4c4b-b68c-efdb5de618b5"
-          (reference "R2") (unit 1)
+          (reference "R7") (unit 1)
         )
       )
@@
   (symbol (lib_id "Device:R") (at 69.85 77.47 0) (unit 1)
     (in_bom yes) (on_board yes) (dnp no)
-    (property "Reference" "R1" (at 69.85 85.09 0)
+    (property "Reference" "R6" (at 69.85 85.09 0)
       (effects (font (size 1.27 1.27)))
     )
@@
       (project "b1"
         (path "/d6142fa5-2354-4512-9919-37616259c364/15951702-f191-4c4b-b68c-efdb5de618b5"
-          (reference "R1") (unit 1)
+          (reference "R6") (unit 1)
         )
       )
@@
   (symbol (lib_id "power:GND") (at 64.77 85.09 0) (unit 1)
     (in_bom yes) (on_board yes) (dnp no) (fields_autoplaced)
-    (property "Reference" "#PWR023" (at 64.77 91.44 0)
+    (property "Reference" "#PWR07" (at 64.77 91.44 0)
       (effects (font (size 1.27 1.27)) hide)
     )
@@
       (project "b1"
         (path "/d6142fa5-2354-4512-9919-37616259c364/15951702-f191-4c4b-b68c-efdb5de618b5"
-          (reference "#PWR023") (unit 1)
+          (reference "#PWR07") (unit 1)
         )
       )
@@
   (symbol (lib_id "74xx:74HC165") (at 116.84 66.04 0) (unit 1)
     (in_bom yes) (on_board yes) (dnp no) (fields_autoplaced)
-    (property "Reference" "U2" (at 119.0341 43.18 0)
+    (property "Reference" "U3" (at 119.0341 43.18 0)
       (effects (font (size 1.27 1.27)) (justify left))
     )
@@
       (project "b1"
         (path "/d6142fa5-2354-4512-9919-37616259c364/15951702-f191-4c4b-b68c-efdb5de618b5"
-          (reference "U2") (unit 1)
+          (reference "U3") (unit 1)
         )
       )
@@
   (symbol (lib_id "Device:R") (at 81.28 77.47 0) (unit 1)
     (in_bom yes) (on_board yes) (dnp no)
-    (property "Reference" "R4" (at 81.28 85.09 0)
+    (property "Reference" "R9" (at 81.28 85.09 0)
       (effects (font (size 1.27 1.27)))
     )
@@
       (project "b1"
         (path "/d6142fa5-2354-4512-9919-37616259c364/15951702-f191-4c4b-b68c-efdb5de618b5"
-          (reference "R4") (unit 1)
+          (reference "R9") (unit 1)
         )
       )
@@
   (symbol (lib_id "Device:R") (at 77.47 77.47 0) (unit 1)
     (in_bom yes) (on_board yes) (dnp no)
-    (property "Reference" "R3" (at 77.47 85.09 0)
+    (property "Reference" "R8" (at 77.47 85.09 0)
       (effects (font (size 1.27 1.27)))
     )
@@
       (project "b1"
         (path "/d6142fa5-2354-4512-9919-37616259c364/15951702-f191-4c4b-b68c-efdb5de618b5"
-          (reference "R3") (unit 1)
-        )
-      )
+          (reference "R8") (unit 1)
+        )
+      )

Commit message: Added more capacitance to the ISR.
Parts:
- added C22: 10u, symbol Device:C_Polarized
Connections:
- net GND: now also C22.2
- net VCC: now also C22.1
Changed lines of the file:
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@@
   (junction (at 50.8 58.42) (diameter 0) (color 0 0 0 0)
   )
+  (junction (at 160.02 41.91) (diameter 0) (color 0 0 0 0)
+  )
   (junction (at 77.47 82.55) (diameter 0) (color 0 0 0 0)
   )
@@
   )
   (junction (at 92.71 68.58) (diameter 0) (color 0 0 0 0)
+  )
+  (junction (at 144.78 31.75) (diameter 0) (color 0 0 0 0)
   )
   (junction (at 88.9 66.04) (diameter 0) (color 0 0 0 0)
@@
     (stroke (width 0) (type default))
   )
+  (wire (pts (xy 160.02 41.91) (xy 144.78 41.91))
+    (stroke (width 0) (type default))
+  )
   (wire (pts (xy 85.09 63.5) (xy 104.14 63.5))
     (stroke (width 0) (type default))
@@
     (stroke (width 0) (type default))
   )
+  (wire (pts (xy 160.02 33.02) (xy 160.02 31.75))
+    (stroke (width 0) (type default))
+  )
   (wire (pts (xy 69.85 53.34) (xy 69.85 73.66))
     (stroke (width 0) (type default))
@@
     (stroke (width 0) (type default))
   )
+  (wire (pts (xy 160.02 40.64) (xy 160.02 41.91))
+    (stroke (width 0) (type default))
+  )
   (wire (pts (xy 88.9 82.55) (xy 88.9 81.28))
     (stroke (width 0) (type default))
@@
     (stroke (width 0) (type default))
   )
-  (wire (pts (xy 144.78 43.18) (xy 144.78 41.91))
+  (wire (pts (xy 160.02 43.18) (xy 160.02 41.91))
     (stroke (width 0) (type default))
   )
@@
   )
   (wire (pts (xy 96.52 71.12) (xy 96.52 73.66))
+    (stroke (width 0) (type default))
+  )
+  (wire (pts (xy 160.02 31.75) (xy 144.78 31.75))
     (stroke (width 0) (type default))
   )
@@
     )
   )
-  (symbol (lib_id "power:GND") (at 144.78 43.18 0) (unit 1)
+  (symbol (lib_id "Device:C_Polarized") (at 160.02 36.83 0) (unit 1)
+    (in_bom yes) (on_board yes) (dnp no)
+    (property "Reference" "C22" (at 163.83 35.56 0)
+      (effects (font (size 1.27 1.27)) (justify left))
+    )
+    (property "Value" "10u" (at 163.83 38.1 0)
+      (effects (font (size 1.27 1.27)) (justify left))
+    )
+    (property "Footprint" "" (at 160.9852 40.64 0)
+      (effects (font (size 1.27 1.27)) hide)
+    )
+    (property "Datasheet" "~" (at 160.02 36.83 0)
+      (effects (font (size 1.27 1.27)) hide)
+    )
+    (pin "2")
+    (pin "1")
+    (instances
+      (project "b1"
+        (path "/d6142fa5-2354-4512-9919-37616259c364/15951702-f191-4c4b-b68c-efdb5de618b5"
+          (reference "C22") (unit 1)
+        )
+      )
+    )
+  )
+  (symbol (lib_id "power:GND") (at 160.02 43.18 0) (unit 1)
     (in_bom yes) (on_board yes) (dnp no) (fields_autoplaced)
-    (property "Reference" "#PWR09" (at 144.78 49.53 0)
-      (effects (font (size 1.27 1.27)) hide)
-    )
-    (property "Value" "GND" (at 144.78 48.26 0)
-      (effects (font (size 1.27 1.27)))
-    )
-    (property "Footprint" "" (at 144.78 43.18 0)
-      (effects (font (size 1.27 1.27)) hide)
-    )
-    (property "Datasheet" "" (at 144.78 43.18 0)
-      (effects (font (size 1.27 1.27)) hide)
-    )
+    (property "Reference" "#PWR09" (at 160.02 49.53 0)
+      (effects (font (size 1.27 1.27)) hide)
+    )
+    (property "Value" "GND" (at 160.02 48.26 0)
+      (effects (font (size 1.27 1.27)))
+    )
+    (property "Footprint" "" (at 160.02 43.18 0)
+      (effects (font (size 1.27 1.27)) hide)
+    )
+    (property "Datasheet" "" (at 160.02 43.18 0)
+      (effects (font (size 1.27 1.27)) hide)
+    )

Commit message: Added diode to prevent ISR from sinking other SPI MISO signals.
Parts:
- added D9: 1N4007, Diode_THT:D_DO-41_SOD81_P10.16mm_Horizontal, symbol Diode:1N4007
Connections:
- net Q7: now also D9.1 (K); no longer U3.9 (Q7)
- new net: D9.2 (A), U3.9 (Q7)
Changed lines of the file:
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@@
+    (stroke (width 0) (type default))
+  )
+  (wire (pts (xy 134.62 50.8) (xy 129.54 50.8))
     (stroke (width 0) (type default))
   )
@@
     (effects (font (size 1.27 1.27)) (justify right))
   )
-  (hierarchical_label "Q7" (shape output) (at 129.54 50.8 0) (fields_autoplaced)
+  (hierarchical_label "Q7" (shape output) (at 142.24 50.8 0) (fields_autoplaced)
     (effects (font (size 1.27 1.27)) (justify left))
   )
@@
         )
       )
+    )
+  )
+  (symbol (lib_id "Diode:1N4007") (at 138.43 50.8 180) (unit 1)
+    (in_bom yes) (on_board yes) (dnp no)
+    (property "Reference" "D9" (at 138.43 48.26 0)
+      (effects (font (size 1.27 1.27)))
+    )
+    (property "Value" "1N4007" (at 138.43 53.34 0)
+      (effects (font (size 1.27 1.27)))
+    )
+    (property "Footprint" "Diode_THT:D_DO-41_SOD81_P10.16mm_Horizontal" (at 138.43 46.355 0)
+      (effects (font (size 1.27 1.27)) hide)
+    )
+    (property "Datasheet" "http://www.vishay.com/docs/88503/1n4001.pdf" (at 138.43 50.8 0)
+      (effects (font (size 1.27 1.27)) hide)
+    )
+    (property "Sim.Device" "D" (at 138.43 50.8 0)
+      (effects (font (size 1.27 1.27)) hide)
+    )
+    (property "Sim.Pins" "1=K 2=A" (at 138.43 50.8 0)
+      (effects (font (size 1.27 1.27)) hide)
+    )
+    (pin "2")
+    (pin "1")
+    (instances
+      (project "b1"
+        (path "/d6142fa5-2354-4512-9919-37616259c364/15951702-f191-4c4b-b68c-efdb5de618b5"
+          (reference "D9") (unit 1)
+        )
+      )

Commit message: Updated schematic to reflect manually shifting in ISR.
Parts:
- removed D9: 1N4007, Diode_THT:D_DO-41_SOD81_P10.16mm_Horizontal, symbol Diode:1N4007
Connections:
- net Q7: now also U3.9 (Q7)
Changed lines of the file:
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@@
-    (stroke (width 0) (type default))
-  )
-  (wire (pts (xy 134.62 50.8) (xy 129.54 50.8))
     (stroke (width 0) (type default))
   )
@@
     (effects (font (size 1.27 1.27)) (justify right))
   )
-  (hierarchical_label "Q7" (shape output) (at 142.24 50.8 0) (fields_autoplaced)
+  (hierarchical_label "Q7" (shape output) (at 129.54 50.8 0) (fields_autoplaced)
     (effects (font (size 1.27 1.27)) (justify left))
   )
@@
         )
       )
-    )
-  )
-  (symbol (lib_id "Diode:1N4007") (at 138.43 50.8 180) (unit 1)
-    (in_bom yes) (on_board yes) (dnp no)
-    (property "Reference" "D9" (at 138.43 48.26 0)
-      (effects (font (size 1.27 1.27)))
-    )
-    (property "Value" "1N4007" (at 138.43 53.34 0)
-      (effects (font (size 1.27 1.27)))
-    )
-    (property "Footprint" "Diode_THT:D_DO-41_SOD81_P10.16mm_Horizontal" (at 138.43 46.355 0)
-      (effects (font (size 1.27 1.27)) hide)
-    )
-    (property "Datasheet" "http://www.vishay.com/docs/88503/1n4001.pdf" (at 138.43 50.8 0)
-      (effects (font (size 1.27 1.27)) hide)
-    )
-    (property "Sim.Device" "D" (at 138.43 50.8 0)
-      (effects (font (size 1.27 1.27)) hide)
-    )
-    (property "Sim.Pins" "1=K 2=A" (at 138.43 50.8 0)
-      (effects (font (size 1.27 1.27)) hide)
-    )
-    (pin "2")
-    (pin "1")
-    (instances
-      (project "b1"
-        (path "/d6142fa5-2354-4512-9919-37616259c364/15951702-f191-4c4b-b68c-efdb5de618b5"
-          (reference "D9") (unit 1)
-        )
-      )
