File: schematics/b1/scanner.kicad_sch (KiCad schematic)
At the start: 0 parts

Commit message: Added schematic page for the status block.
Other:
- company: (none) -> shawnd.xyz
Changed lines of the file:
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@@
   (title_block
     (title "B1")
-    (date "2024-02-01")
+    (date "2024-02-05")
     (rev "1")
+    (company "shawnd.xyz")
     (comment 2 "scanning as well as radio communications and outputs/displays.")
     (comment 3 "A B1 (Badger One) node is the core hardware unit of the Badger sytem. It handles card")

Commit message: Added schematic page for scanner.
Parts:
- added P1: RFID-RC522, symbol RC522:RFID-RC522-MODULE
Connections:
- new net GND: P1.6 (GND)
- new net MISO: P1.4 (MISO)
- new net MOSI: P1.3 (MOSI)
- new net RST: P1.7 (RST)
- new net SCK: P1.2 (SCK)
- new net SDA: P1.1 (SDA)
- new net VCC: P1.8 (3.3V)
- no-connect marks 0 -> 1
Other:
- title: B1 -> Scanner
Changed lines of the file:
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@@
 (kicad_sch (version 20230121) (generator eeschema)
-  (paper "A4")
+  (paper "A5")
   (title_block
-    (title "B1")
+    (title "Scanner")
     (date "2024-02-05")
     (rev "1")
     (company "shawnd.xyz")
-    (comment 2 "scanning as well as radio communications and outputs/displays.")
-    (comment 3 "A B1 (Badger One) node is the core hardware unit of the Badger sytem. It handles card")
+    (comment 2 "enclosure for better scanning ability.")
+    (comment 3 "Detaching it from the motherboard allows it to be placed closer to the surface of the")
+    (comment 4 "The scanner is an RFID-RC522 module attached to the motherboard via a ribbon cable.")
+  )
+  (no_connect (at 110.49 58.42))
+  (hierarchical_label "VCC" (shape input) (at 99.06 50.8 90) (fields_autoplaced)
+    (effects (font (size 1.27 1.27)) (justify left))
+  )
+  (hierarchical_label "MOSI" (shape input) (at 88.9 60.96 180) (fields_autoplaced)
+    (effects (font (size 1.27 1.27)) (justify right))
+  )
+  (hierarchical_label "SDA" (shape input) (at 88.9 55.88 180) (fields_autoplaced)
+    (effects (font (size 1.27 1.27)) (justify right))
+  )
+  (hierarchical_label "SCK" (shape input) (at 88.9 58.42 180) (fields_autoplaced)
+    (effects (font (size 1.27 1.27)) (justify right))
+  )
+  (hierarchical_label "RST" (shape input) (at 88.9 63.5 180) (fields_autoplaced)
+    (effects (font (size 1.27 1.27)) (justify right))
+  )
+  (hierarchical_label "MISO" (shape output) (at 110.49 55.88 0) (fields_autoplaced)
+    (effects (font (size 1.27 1.27)) (justify left))
+  )
+  (symbol (lib_id "RC522:RFID-RC522-MODULE") (at 107.95 80.01 0) (unit 1)
+    (in_bom yes) (on_board yes) (dnp no) (fields_autoplaced)
+    (property "Reference" "P1" (at 101.6 48.26 0)
+      (effects (font (size 1.524 1.524)) (justify left))
+    )
+    (property "Value" "RFID-RC522" (at 101.6 50.8 0)
+      (effects (font (size 1.524 1.524)) (justify left))
+    )
+    (property "Footprint" "" (at 125.095 70.485 90)
+      (effects (font (size 1.524 1.524)))
+    )
+    (property "Datasheet" "" (at 125.095 70.485 90)
+      (effects (font (size 1.524 1.524)))
+    )
+    (pin "8")
+    (pin "1")
+    (pin "3")
+    (pin "5")
+    (pin "4")
+    (pin "7")
+    (pin "6")
+    (pin "2")
+    (instances
+      (project "b1"
+        (path "/d6142fa5-2354-4512-9919-37616259c364/64a24a3a-7315-4dfd-86dd-98547cdfac2f"
+          (reference "P1") (unit 1)
+        )
+        (path "/d6142fa5-2354-4512-9919-37616259c364/fdcf7d10-3243-4165-8310-96b25d91ab12"
+          (reference "P1") (unit 1)
+        )
+      )
+    )
+  )
+  (symbol (lib_id "power:GND") (at 99.06 68.58 0) (unit 1)
+    (in_bom yes) (on_board yes) (dnp no) (fields_autoplaced)
+    (property "Reference" "#PWR021" (at 99.06 74.93 0)
+      (effects (font (size 1.27 1.27)) hide)
+    )
+    (property "Value" "GND" (at 99.06 73.66 0)
+      (effects (font (size 1.27 1.27)))
+    )
+    (property "Footprint" "" (at 99.06 68.58 0)
+      (effects (font (size 1.27 1.27)) hide)
+    )
+    (property "Datasheet" "" (at 99.06 68.58 0)
+      (effects (font (size 1.27 1.27)) hide)
+    )
+    (pin "1")
+    (instances
+      (project "b1"
+        (path "/d6142fa5-2354-4512-9919-37616259c364/64a24a3a-7315-4dfd-86dd-98547cdfac2f"
+          (reference "#PWR021") (unit 1)
+        )
+      )
+    )
   )
 )

Commit message: Updated schematics.
Other:
- note added: "A bypass capacitor is not needed as the module itself has its own onboard."
Changed lines of the file:
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@@
   )
   (no_connect (at 110.49 58.42))
+  (text "A bypass capacitor is not needed\nas the module itself has its own\nonboard."
+    (at 120.65 59.69 0)
+    (effects (font (size 1.27 1.27)) (justify left bottom))
+  )
   (hierarchical_label "VCC" (shape input) (at 99.06 50.8 90) (fields_autoplaced)
     (effects (font (size 1.27 1.27)) (justify left))
@@
           (reference "P1") (unit 1)
         )
-        (path "/d6142fa5-2354-4512-9919-37616259c364/fdcf7d10-3243-4165-8310-96b25d91ab12"
-          (reference "P1") (unit 1)
-        )

Commit message: Updated bypass capacitor values.
Other:
- note added: "Bypass capacitors are not needed as the module itself has its own onboard."
- note removed: "A bypass capacitor is not needed as the module itself has its own onboard."
Changed lines of the file:
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@@
   )
   (no_connect (at 110.49 58.42))
-  (text "A bypass capacitor is not needed\nas the module itself has its own\nonboard."
+  (text "Bypass capacitors are not needed\nas the module itself has its own\nonboard."
     (at 120.65 59.69 0)
     (effects (font (size 1.27 1.27)) (justify left bottom))

Commit message: Updated labels.
Connections:
- net SCK renamed ~{SS}
Changed lines of the file:
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@@
     (effects (font (size 1.27 1.27)) (justify right))
   )
-  (hierarchical_label "SCK" (shape input) (at 88.9 58.42 180) (fields_autoplaced)
+  (hierarchical_label "~{SS}" (shape input) (at 88.9 58.42 180) (fields_autoplaced)
     (effects (font (size 1.27 1.27)) (justify right))
   )

Commit message: General schematic updates.
Connections:
- net SDA is gone; now on net ~{SS}: P1.1 (SDA)
- net ~{SS}: no longer P1.2 (SCK)
- new net SCK: P1.2 (SCK)
Changed lines of the file:
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@@
     (effects (font (size 1.27 1.27)) (justify right))
   )
-  (hierarchical_label "SDA" (shape input) (at 88.9 55.88 180) (fields_autoplaced)
+  (hierarchical_label "~{SS}" (shape input) (at 88.9 55.88 180) (fields_autoplaced)
     (effects (font (size 1.27 1.27)) (justify right))
   )
-  (hierarchical_label "~{SS}" (shape input) (at 88.9 58.42 180) (fields_autoplaced)
+  (hierarchical_label "SCK" (shape input) (at 88.9 58.42 180) (fields_autoplaced)
     (effects (font (size 1.27 1.27)) (justify right))
   )
@@
   (symbol (lib_id "power:GND") (at 99.06 68.58 0) (unit 1)
     (in_bom yes) (on_board yes) (dnp no) (fields_autoplaced)
-    (property "Reference" "#PWR021" (at 99.06 74.93 0)
+    (property "Reference" "#PWR022" (at 99.06 74.93 0)
       (effects (font (size 1.27 1.27)) hide)
     )
@@
       (project "b1"
         (path "/d6142fa5-2354-4512-9919-37616259c364/64a24a3a-7315-4dfd-86dd-98547cdfac2f"
-          (reference "#PWR021") (unit 1)
+          (reference "#PWR022") (unit 1)
         )
       )
