File: schematics/b1/scanner.kicad_sch (KiCad schematic)
At the start: 6 parts, among them P1 RFID-RC522

Commit message: Updated annotations.
Parts:
- renumbered C7 to C25, TP21 to TP37, TP44 to TP38, TP31 to TP39, TP22 to TP40
Changed lines of the file:
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@@
   (symbol (lib_id "Connector:TestPoint") (at 74.93 64.77 180) (unit 1)
     (in_bom yes) (on_board yes) (dnp no)
-    (property "Reference" "TP44" (at 73.66 69.85 90)
+    (property "Reference" "TP38" (at 74.93 69.85 90)
       (effects (font (size 1.27 1.27)) (justify left))
     )
     (property "Value" "TestPoint" (at 76.2 69.85 90)
-      (effects (font (size 1.27 1.27)) (justify left))
+      (effects (font (size 1.27 1.27)) (justify left) hide)
     )
     (property "Footprint" "" (at 69.85 64.77 0)
@@
       (project "b1"
         (path "/d6142fa5-2354-4512-9919-37616259c364/64a24a3a-7315-4dfd-86dd-98547cdfac2f"
-          (reference "TP44") (unit 1)
+          (reference "TP38") (unit 1)
         )
       )
@@
   (symbol (lib_id "power:GND") (at 99.06 71.12 0) (unit 1)
     (in_bom yes) (on_board yes) (dnp no) (fields_autoplaced)
-    (property "Reference" "#PWR018" (at 99.06 77.47 0)
+    (property "Reference" "#PWR036" (at 99.06 77.47 0)
       (effects (font (size 1.27 1.27)) hide)
     )
@@
       (project "b1"
         (path "/d6142fa5-2354-4512-9919-37616259c364/64a24a3a-7315-4dfd-86dd-98547cdfac2f"
-          (reference "#PWR018") (unit 1)
+          (reference "#PWR036") (unit 1)
         )
       )
@@
   (symbol (lib_id "Device:C_Polarized") (at 87.63 39.37 0) (unit 1)
     (in_bom yes) (on_board yes) (dnp no)
-    (property "Reference" "C7" (at 91.44 38.1 0)
+    (property "Reference" "C25" (at 91.44 38.1 0)
       (effects (font (size 1.27 1.27)) (justify left))
     )
@@
       (project "b1"
         (path "/d6142fa5-2354-4512-9919-37616259c364/64a24a3a-7315-4dfd-86dd-98547cdfac2f"
-          (reference "C7") (unit 1)
+          (reference "C25") (unit 1)
         )
       )
@@
   (symbol (lib_id "power:GND") (at 87.63 43.18 0) (unit 1)
     (in_bom yes) (on_board yes) (dnp no)
-    (property "Reference" "#PWR017" (at 87.63 49.53 0)
+    (property "Reference" "#PWR035" (at 87.63 49.53 0)
       (effects (font (size 1.27 1.27)) hide)
     )
@@
       (project "b1"
         (path "/d6142fa5-2354-4512-9919-37616259c364/64a24a3a-7315-4dfd-86dd-98547cdfac2f"
-          (reference "#PWR017") (unit 1)
+          (reference "#PWR035") (unit 1)
         )
       )
@@
   (symbol (lib_id "Connector:TestPoint") (at 85.09 64.77 180) (unit 1)
     (in_bom yes) (on_board yes) (dnp no)
-    (property "Reference" "TP31" (at 83.82 69.85 90)
+    (property "Reference" "TP39" (at 85.09 69.85 90)
       (effects (font (size 1.27 1.27)) (justify left))
     )
     (property "Value" "TestPoint" (at 86.36 69.85 90)
-      (effects (font (size 1.27 1.27)) (justify left))
+      (effects (font (size 1.27 1.27)) (justify left) hide)
     )
     (property "Footprint" "" (at 80.01 64.77 0)
@@
       (project "b1"
         (path "/d6142fa5-2354-4512-9919-37616259c364/64a24a3a-7315-4dfd-86dd-98547cdfac2f"
-          (reference "TP31") (unit 1)
+          (reference "TP39") (unit 1)
         )
       )
@@
   )
   (symbol (lib_id "Connector:TestPoint") (at 100.33 41.91 270) (unit 1)
-    (in_bom yes) (on_board yes) (dnp no) (fields_autoplaced)
-    (property "Reference" "TP21" (at 105.41 40.64 90)
+    (in_bom yes) (on_board yes) (dnp no)
+    (property "Reference" "TP37" (at 105.41 41.91 90)
       (effects (font (size 1.27 1.27)) (justify left))
     )
     (property "Value" "TestPoint" (at 105.41 43.18 90)
-      (effects (font (size 1.27 1.27)) (justify left))
+      (effects (font (size 1.27 1.27)) (justify left) hide)
     )
     (property "Footprint" "" (at 100.33 46.99 0)
@@
       (project "b1"
         (path "/d6142fa5-2354-4512-9919-37616259c364/64a24a3a-7315-4dfd-86dd-98547cdfac2f"
-          (reference "TP21") (unit 1)
+          (reference "TP37") (unit 1)
         )
       )
@@
   )
   (symbol (lib_id "Connector:TestPoint") (at 100.33 69.85 270) (unit 1)
-    (in_bom yes) (on_board yes) (dnp no) (fields_autoplaced)
-    (property "Reference" "TP22" (at 105.41 68.58 90)
+    (in_bom yes) (on_board yes) (dnp no)
+    (property "Reference" "TP40" (at 105.41 69.85 90)
       (effects (font (size 1.27 1.27)) (justify left))
     )
     (property "Value" "TestPoint" (at 105.41 71.12 90)
-      (effects (font (size 1.27 1.27)) (justify left))
+      (effects (font (size 1.27 1.27)) (justify left) hide)
     )
     (property "Footprint" "" (at 100.33 74.93 0)
@@
       (project "b1"
         (path "/d6142fa5-2354-4512-9919-37616259c364/64a24a3a-7315-4dfd-86dd-98547cdfac2f"
-          (reference "TP22") (unit 1)
+          (reference "TP40") (unit 1)
         )
       )
