File: schematics/b1/scanner.kicad_sch (KiCad schematic)
At the start: 6 parts, among them P1 RFID-RC522

Commit message: Assigned some footprints.
Parts:
- C25: footprint (none) -> Capacitor_THT:CP_Radial_D8.0mm_P3.80mm
- P1: footprint (none) -> Connector_PinHeader_2.54mm:PinHeader_1x08_P2.54mm_Vertical
Changed lines of the file:
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@@
       (effects (font (size 1.524 1.524)) (justify left))
     )
-    (property "Footprint" "" (at 125.095 70.485 90)
-      (effects (font (size 1.524 1.524)))
+    (property "Footprint" "Connector_PinHeader_2.54mm:PinHeader_1x08_P2.54mm_Vertical" (at 125.095 70.485 90)
+      (effects (font (size 1.524 1.524)) hide)
     )
     (property "Datasheet" "" (at 125.095 70.485 90)
@@
       (effects (font (size 1.27 1.27)) (justify left))
     )
-    (property "Footprint" "" (at 88.5952 43.18 0)
+    (property "Footprint" "Capacitor_THT:CP_Radial_D8.0mm_P3.80mm" (at 88.5952 43.18 0)
       (effects (font (size 1.27 1.27)) hide)
     )

Commit message: Finished assigning footprints.
Parts:
- TP37, TP38, TP39, TP40: footprint (none) -> TestPoint:TestPoint_Loop_D2.50mm_Drill1.0mm
Changed lines of the file:
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@@
       (effects (font (size 1.27 1.27)) (justify left) hide)
     )
-    (property "Footprint" "" (at 69.85 64.77 0)
+    (property "Footprint" "TestPoint:TestPoint_Loop_D2.50mm_Drill1.0mm" (at 69.85 64.77 0)
       (effects (font (size 1.27 1.27)) hide)
     )
@@
       (effects (font (size 1.27 1.27)) (justify left) hide)
     )
-    (property "Footprint" "" (at 80.01 64.77 0)
+    (property "Footprint" "TestPoint:TestPoint_Loop_D2.50mm_Drill1.0mm" (at 80.01 64.77 0)
       (effects (font (size 1.27 1.27)) hide)
     )
@@
       (effects (font (size 1.27 1.27)) (justify left) hide)
     )
-    (property "Footprint" "" (at 100.33 46.99 0)
+    (property "Footprint" "TestPoint:TestPoint_Loop_D2.50mm_Drill1.0mm" (at 100.33 46.99 0)
       (effects (font (size 1.27 1.27)) hide)
     )
@@
       (effects (font (size 1.27 1.27)) (justify left) hide)
     )
-    (property "Footprint" "" (at 100.33 74.93 0)
+    (property "Footprint" "TestPoint:TestPoint_Loop_D2.50mm_Drill1.0mm" (at 100.33 74.93 0)
       (effects (font (size 1.27 1.27)) hide)
     )
