File: schematics/b1/wifi.kicad_sch (KiCad schematic)
At the start: 13 parts, among them J1 SERIAL, SW2 RESET, SW3 BOOT, SW4 JUMP, U4 L7805, U6 ESP-12F

Commit message: Updated annotations.
Parts:
- renumbered C18 to C1, D8 to D1, R26 to R1, R27 to R2, R30 to R3, R29 to R4, R28 to R5, SW4 to SW1, U4 to U1, U6 to U2
Other:
- moved on the sheet: R5
Changed lines of the file:
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@@
   (title_block
     (title "B1")
-    (date "2024-02-06")
+    (date "2024-02-15")
     (rev "1")
     (company "shawnd.xyz")
@@
     (stroke (width 0) (type default))
   )
-  (wire (pts (xy 149.86 64.77) (xy 149.86 66.04))
+  (wire (pts (xy 149.86 62.23) (xy 149.86 66.04))
     (stroke (width 0) (type default))
   )
@@
     (effects (font (size 1.27 1.27)) (justify left))
   )
-  (hierarchical_label "VCC" (shape input) (at 149.86 57.15 90) (fields_autoplaced)
+  (hierarchical_label "VCC" (shape input) (at 149.86 54.61 90) (fields_autoplaced)
     (effects (font (size 1.27 1.27)) (justify left))
   )
@@
   (symbol (lib_id "Device:R") (at 88.9 63.5 90) (unit 1)
     (in_bom yes) (on_board yes) (dnp no)
-    (property "Reference" "R27" (at 88.9 60.96 90)
+    (property "Reference" "R2" (at 88.9 60.96 90)
       (effects (font (size 1.27 1.27)))
     )
@@
       (project "b1"
         (path "/d6142fa5-2354-4512-9919-37616259c364/a74f58bd-54a1-4bdf-85a5-bb477b4492d8"
-          (reference "R27") (unit 1)
+          (reference "R2") (unit 1)
         )
       )
@@
   (symbol (lib_id "Device:R") (at 72.39 53.34 180) (unit 1)
     (in_bom yes) (on_board yes) (dnp no)
-    (property "Reference" "R26" (at 69.85 52.07 0)
+    (property "Reference" "R1" (at 69.85 52.07 0)
       (effects (font (size 1.27 1.27)) (justify left))
     )
@@
       (project "b1"
         (path "/d6142fa5-2354-4512-9919-37616259c364/a74f58bd-54a1-4bdf-85a5-bb477b4492d8"
-          (reference "R26") (unit 1)
+          (reference "R1") (unit 1)
         )
       )
@@
   (symbol (lib_id "power:GND") (at 130.81 91.44 0) (unit 1)
     (in_bom yes) (on_board yes) (dnp no) (fields_autoplaced)
-    (property "Reference" "#PWR030" (at 130.81 97.79 0)
+    (property "Reference" "#PWR04" (at 130.81 97.79 0)
       (effects (font (size 1.27 1.27)) hide)
     )
@@
       (project "b1"
         (path "/d6142fa5-2354-4512-9919-37616259c364/a74f58bd-54a1-4bdf-85a5-bb477b4492d8"
-          (reference "#PWR030") (unit 1)
+          (reference "#PWR04") (unit 1)
         )
       )
@@
   (symbol (lib_id "power:GND") (at 93.98 44.45 0) (unit 1)
     (in_bom yes) (on_board yes) (dnp no)
-    (property "Reference" "#PWR026" (at 93.98 50.8 0)
+    (property "Reference" "#PWR02" (at 93.98 50.8 0)
       (effects (font (size 1.27 1.27)) hide)
     )
@@
       (project "b1"
         (path "/d6142fa5-2354-4512-9919-37616259c364/a74f58bd-54a1-4bdf-85a5-bb477b4492d8"
-          (reference "#PWR026") (unit 1)
+          (reference "#PWR02") (unit 1)
         )
       )
@@
   (symbol (lib_id "Diode:1N4007") (at 107.95 27.94 90) (unit 1)
     (in_bom yes) (on_board yes) (dnp no) (fields_autoplaced)
-    (property "Reference" "D8" (at 110.49 26.67 90)
+    (property "Reference" "D1" (at 110.49 26.67 90)
       (effects (font (size 1.27 1.27)) (justify right))
     )
@@
       (project "b1"
         (path "/d6142fa5-2354-4512-9919-37616259c364/a74f58bd-54a1-4bdf-85a5-bb477b4492d8"
-          (reference "D8") (unit 1)
+          (reference "D1") (unit 1)
         )
       )
@@
   (symbol (lib_id "Device:R") (at 130.81 87.63 0) (mirror y) (unit 1)
     (in_bom yes) (on_board yes) (dnp no)
-    (property "Reference" "R30" (at 133.35 86.36 0)
+    (property "Reference" "R3" (at 133.35 86.36 0)
       (effects (font (size 1.27 1.27)) (justify right))
     )
@@
       (project "b1"
         (path "/d6142fa5-2354-4512-9919-37616259c364/a74f58bd-54a1-4bdf-85a5-bb477b4492d8"
-          (reference "R30") (unit 1)
-        )
-      )
-    )
-  )
-  (symbol (lib_id "Device:R") (at 149.86 60.96 0) (unit 1)
-    (in_bom yes) (on_board yes) (dnp no) (fields_autoplaced)
-    (property "Reference" "R28" (at 152.4 59.69 0)
-      (effects (font (size 1.27 1.27)) (justify left))
-    )
-    (property "Value" "10k" (at 152.4 62.23 0)
-      (effects (font (size 1.27 1.27)) (justify left))
-    )
-    (property "Footprint" "" (at 148.082 60.96 90)
-      (effects (font (size 1.27 1.27)) hide)
-    )
-    (property "Datasheet" "~" (at 149.86 60.96 0)
-      (effects (font (size 1.27 1.27)) hide)
-    )
-    (pin "1")
-    (pin "2")
-    (instances
-      (project "b1"
-        (path "/d6142fa5-2354-4512-9919-37616259c364/a74f58bd-54a1-4bdf-85a5-bb477b4492d8"
-          (reference "R28") (unit 1)
+          (reference "R3") (unit 1)
+        )
+      )
+    )
+  )
+  (symbol (lib_id "Device:R") (at 149.86 58.42 0) (unit 1)
+    (in_bom yes) (on_board yes) (dnp no) (fields_autoplaced)
+    (property "Reference" "R5" (at 152.4 57.15 0)
+      (effects (font (size 1.27 1.27)) (justify left))
+    )
+    (property "Value" "10k" (at 152.4 59.69 0)
+      (effects (font (size 1.27 1.27)) (justify left))
+    )
+    (property "Footprint" "" (at 148.082 58.42 90)
+      (effects (font (size 1.27 1.27)) hide)
+    )
+    (property "Datasheet" "~" (at 149.86 58.42 0)
+      (effects (font (size 1.27 1.27)) hide)
+    )
+    (pin "1")
+    (pin "2")
+    (instances
+      (project "b1"
+        (path "/d6142fa5-2354-4512-9919-37616259c364/a74f58bd-54a1-4bdf-85a5-bb477b4492d8"
+          (reference "R5") (unit 1)
         )
       )
@@
   (symbol (lib_id "Switch:SW_Push") (at 67.31 33.02 0) (unit 1)
     (in_bom yes) (on_board yes) (dnp no)
-    (property "Reference" "SW4" (at 67.31 27.94 0)
+    (property "Reference" "SW1" (at 67.31 27.94 0)
       (effects (font (size 1.27 1.27)))
     )
@@
       (project "b1"
         (path "/d6142fa5-2354-4512-9919-37616259c364/a74f58bd-54a1-4bdf-85a5-bb477b4492d8"
-          (reference "SW4") (unit 1)
+          (reference "SW1") (unit 1)
         )
       )
@@
   (symbol (lib_id "power:GND") (at 149.86 77.47 0) (unit 1)
     (in_bom yes) (on_board yes) (dnp no) (fields_autoplaced)
-    (property "Reference" "#PWR03" (at 149.86 83.82 0)
+    (property "Reference" "#PWR06" (at 149.86 83.82 0)
       (effects (font (size 1.27 1.27)) hide)
     )
@@
       (project "b1"
         (path "/d6142fa5-2354-4512-9919-37616259c364/a74f58bd-54a1-4bdf-85a5-bb477b4492d8"
-          (reference "#PWR03") (unit 1)
+          (reference "#PWR06") (unit 1)
         )
       )
@@
   (symbol (lib_id "Regulator_Linear:L7805") (at 80.01 33.02 0) (unit 1)
     (in_bom yes) (on_board yes) (dnp no) (fields_autoplaced)
-    (property "Reference" "U4" (at 80.01 26.67 0)
+    (property "Reference" "U1" (at 80.01 26.67 0)
       (effects (font (size 1.27 1.27)))
     )
@@
       (project "b1"
         (path "/d6142fa5-2354-4512-9919-37616259c364/a74f58bd-54a1-4bdf-85a5-bb477b4492d8"
-          (reference "U4") (unit 1)
+          (reference "U1") (unit 1)
         )
       )
@@
   (symbol (lib_id "power:GND") (at 72.39 69.85 0) (unit 1)
     (in_bom yes) (on_board yes) (dnp no) (fields_autoplaced)
-    (property "Reference" "#PWR027" (at 72.39 76.2 0)
+    (property "Reference" "#PWR01" (at 72.39 76.2 0)
       (effects (font (size 1.27 1.27)) hide)
     )
@@
       (project "b1"
         (path "/d6142fa5-2354-4512-9919-37616259c364/a74f58bd-54a1-4bdf-85a5-bb477b4492d8"
-          (reference "#PWR027") (unit 1)
+          (reference "#PWR01") (unit 1)
         )
       )
@@
   (symbol (lib_id "power:GND") (at 135.89 38.1 0) (unit 1)
     (in_bom yes) (on_board yes) (dnp no)
-    (property "Reference" "#PWR029" (at 135.89 44.45 0)
+    (property "Reference" "#PWR05" (at 135.89 44.45 0)
       (effects (font (size 1.27 1.27)) hide)
     )
@@
       (project "b1"
         (path "/d6142fa5-2354-4512-9919-37616259c364/a74f58bd-54a1-4bdf-85a5-bb477b4492d8"
-          (reference "#PWR029") (unit 1)
+          (reference "#PWR05") (unit 1)
         )
       )
@@
   (symbol (lib_id "Device:R") (at 139.7 58.42 180) (unit 1)
     (in_bom yes) (on_board yes) (dnp no)
-    (property "Reference" "R29" (at 142.24 57.15 0)
+    (property "Reference" "R4" (at 142.24 57.15 0)
       (effects (font (size 1.27 1.27)) (justify right))
     )
@@
       (project "b1"
         (path "/d6142fa5-2354-4512-9919-37616259c364/a74f58bd-54a1-4bdf-85a5-bb477b4492d8"
-          (reference "R29") (unit 1)
+          (reference "R4") (unit 1)
         )
       )
@@
   (symbol (lib_id "RF_Module:ESP-12F") (at 107.95 73.66 0) (unit 1)
     (in_bom yes) (on_board yes) (dnp no) (fields_autoplaced)
-    (property "Reference" "U6" (at 110.1441 50.8 0)
+    (property "Reference" "U2" (at 110.1441 50.8 0)
       (effects (font (size 1.27 1.27)) (justify left))
     )
@@
       (project "b1"
         (path "/d6142fa5-2354-4512-9919-37616259c364/a74f58bd-54a1-4bdf-85a5-bb477b4492d8"
-          (reference "U6") (unit 1)
+          (reference "U2") (unit 1)
         )
       )
@@
   (symbol (lib_id "Device:C_Polarized") (at 93.98 38.1 0) (unit 1)
     (in_bom yes) (on_board yes) (dnp no)
-    (property "Reference" "C18" (at 97.79 35.941 0)
+    (property "Reference" "C1" (at 97.79 35.941 0)
       (effects (font (size 1.27 1.27)) (justify left))
     )
@@
       (project "b1"
         (path "/d6142fa5-2354-4512-9919-37616259c364/a74f58bd-54a1-4bdf-85a5-bb477b4492d8"
-          (reference "C18") (unit 1)
+          (reference "C1") (unit 1)
         )
       )
@@
   (symbol (lib_id "power:GND") (at 107.95 91.44 0) (unit 1)
     (in_bom yes) (on_board yes) (dnp no) (fields_autoplaced)
-    (property "Reference" "#PWR028" (at 107.95 97.79 0)
+    (property "Reference" "#PWR03" (at 107.95 97.79 0)
       (effects (font (size 1.27 1.27)) hide)
     )
@@
       (project "b1"
         (path "/d6142fa5-2354-4512-9919-37616259c364/a74f58bd-54a1-4bdf-85a5-bb477b4492d8"
-          (reference "#PWR028") (unit 1)
-        )
-      )
+          (reference "#PWR03") (unit 1)
+        )
+      )
