File: schematics/b1/lora.kicad_sch (KiCad schematic)
At the start: 10 parts, among them U7 Ai-Thinker-Ra-02

Commit message: Assigned some footprints.
Parts:
- C26: footprint (none) -> Capacitor_THT:CP_Radial_D8.0mm_P3.80mm
- C27: footprint (none) -> Capacitor_THT:CP_Radial_D4.0mm_P2.00mm
- C28, C29: footprint (none) -> Capacitor_SMD:C_1206_3216Metric_Pad1.33x1.80mm_HandSolder
Changed lines of the file:
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@@
       (effects (font (size 1.27 1.27)) (justify left))
     )
-    (property "Footprint" "" (at 88.5952 39.37 0)
+    (property "Footprint" "Capacitor_SMD:C_1206_3216Metric_Pad1.33x1.80mm_HandSolder" (at 88.5952 39.37 0)
       (effects (font (size 1.27 1.27)) hide)
     )
@@
       (effects (font (size 1.27 1.27)) (justify left))
     )
-    (property "Footprint" "" (at 77.1652 39.37 0)
+    (property "Footprint" "Capacitor_SMD:C_1206_3216Metric_Pad1.33x1.80mm_HandSolder" (at 77.1652 39.37 0)
       (effects (font (size 1.27 1.27)) hide)
     )
@@
       (effects (font (size 1.27 1.27)) (justify left))
     )
-    (property "Footprint" "" (at 54.3052 39.37 0)
+    (property "Footprint" "Capacitor_THT:CP_Radial_D8.0mm_P3.80mm" (at 54.3052 39.37 0)
       (effects (font (size 1.27 1.27)) hide)
     )
@@
       (effects (font (size 1.27 1.27)) (justify left))
     )
-    (property "Footprint" "" (at 65.7352 39.37 0)
+    (property "Footprint" "Capacitor_THT:CP_Radial_D4.0mm_P2.00mm" (at 65.7352 39.37 0)
       (effects (font (size 1.27 1.27)) hide)
     )
