File: schematics/b1/bid_register.kicad_sch (KiCad schematic)
At the start: 19 parts, among them SW5 SW_DIP_x08, U5 74HC165

Commit message: Routed traces.
Parts:
- removed TP31: TestPoint, TestPoint:TestPoint_Loop_D2.50mm_Drill1.0mm, symbol Connector:TestPoint
Changed lines of the file:
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@@
   (junction (at 33.02 60.96) (diameter 0) (color 0 0 0 0)
-  )
-  (junction (at 125.73 90.17) (diameter 0) (color 0 0 0 0)
   )
   (junction (at 33.02 63.5) (diameter 0) (color 0 0 0 0)
@@
     (stroke (width 0) (type default))
   )
-  (wire (pts (xy 125.73 90.17) (xy 125.73 88.9))
-    (stroke (width 0) (type default))
-  )
   (wire (pts (xy 52.07 80.01) (xy 52.07 78.74))
     (stroke (width 0) (type default))
@@
     (stroke (width 0) (type default))
   )
-  (wire (pts (xy 127 90.17) (xy 125.73 90.17))
-    (stroke (width 0) (type default))
-  )
   (wire (pts (xy 49.53 50.8) (xy 52.07 50.8))
     (stroke (width 0) (type default))
@@
   )
   (wire (pts (xy 114.3 34.29) (xy 114.3 33.02))
-    (stroke (width 0) (type default))
-  )
-  (wire (pts (xy 125.73 91.44) (xy 125.73 90.17))
     (stroke (width 0) (type default))
   )
@@
         (path "/d6142fa5-2354-4512-9919-37616259c364/15951702-f191-4c4b-b68c-efdb5de618b5"
           (reference "TP30") (unit 1)
-        )
-      )
-    )
-  )
-  (symbol (lib_id "Connector:TestPoint") (at 127 90.17 270) (unit 1)
-    (in_bom yes) (on_board yes) (dnp no)
-    (property "Reference" "TP31" (at 132.08 90.17 90)
-      (effects (font (size 1.27 1.27)) (justify left))
-    )
-    (property "Value" "TestPoint" (at 132.08 91.44 90)
-      (effects (font (size 1.27 1.27)) (justify left) hide)
-    )
-    (property "Footprint" "TestPoint:TestPoint_Loop_D2.50mm_Drill1.0mm" (at 127 95.25 0)
-      (effects (font (size 1.27 1.27)) hide)
-    )
-    (property "Datasheet" "~" (at 127 95.25 0)
-      (effects (font (size 1.27 1.27)) hide)
-    )
-    (pin "1")
-    (instances
-      (project "b1"
-        (path "/d6142fa5-2354-4512-9919-37616259c364/15951702-f191-4c4b-b68c-efdb5de618b5"
-          (reference "TP31") (unit 1)
         )
       )
@@
     )
   )
-  (symbol (lib_id "power:GND") (at 125.73 91.44 0) (unit 1)
-    (in_bom yes) (on_board yes) (dnp no)
-    (property "Reference" "#PWR028" (at 125.73 97.79 0)
-      (effects (font (size 1.27 1.27)) hide)
-    )
-    (property "Value" "GND" (at 125.73 96.52 0)
-      (effects (font (size 1.27 1.27)))
-    )
-    (property "Footprint" "" (at 125.73 91.44 0)
-      (effects (font (size 1.27 1.27)) hide)
-    )
-    (property "Datasheet" "" (at 125.73 91.44 0)
+  (symbol (lib_id "power:GND") (at 125.73 88.9 0) (unit 1)
+    (in_bom yes) (on_board yes) (dnp no)
+    (property "Reference" "#PWR028" (at 125.73 95.25 0)
+      (effects (font (size 1.27 1.27)) hide)
+    )
+    (property "Value" "GND" (at 125.73 93.98 0)
+      (effects (font (size 1.27 1.27)))
+    )
+    (property "Footprint" "" (at 125.73 88.9 0)
+      (effects (font (size 1.27 1.27)) hide)
+    )
+    (property "Datasheet" "" (at 125.73 88.9 0)
       (effects (font (size 1.27 1.27)) hide)
     )
@@
       (effects (font (size 1.27 1.27)) hide)
     )
-    (property "Value" "GND" (at 87.63 40.64 0)
-      (effects (font (size 1.27 1.27)))
-    )
+    (property "Value" "GND" (at 91.44 40.64 0)
+      (effects (font (size 1.27 1.27)))
+    )
